File: nrf54_promicro.kicad_sch (KiCad schematic)
At the start: 60 parts, among them J1 GSB1C4621DS1HR, J2 Conn_01x13_Socket, J3 Conn_01x13_Socket, U1 BQ24075RGT, U2 nRF54L10, U3 TPS62172DSG, U4 AP22913CN4, Y1 32.768k, Y2 32M

Commit message: Continued to improve layout. Updated README.md
Other:
- note added: "B2B Conn."
- note added: "Regulators"
- note added: "Type-C Conn."
- note removed: "Note: See Bypass Page for Bypass Cap Details"
- moved on the sheet: C1, C15, C16, C2, C20, C21, C25, C3, C4, C5, C6, C7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

Commit message: Swapped U4 for lower Iq load switch. Fixed DRCs. Fixed Layout.
Parts:
- removed U4: AP22913CN4, Package_CSP:WLCSP-4-X1-WLB0909-4_0.89x0.89mm_P0.5mm, symbol Power_Management:AP22913CN4
- added U4: TPS22917DBV, Package_TO_SOT_SMD:SOT-23-6, symbol Power_Management:TPS22917DBV
Connections:
- net GND: now also U4.2 (GND)
- net VEXT: now also U4.5 (QOD), U4.6 (VOUT)
- net VSYS: now also U4.1 (VIN)
- net EXT_EN renamed VEXT_DIS_L
- net VEXT_DIS_L: now also U4.3 (ON)
- no-connect marks 13 -> 14
Other:
- moved on the sheet: C20, C21, R12

Commit message: Updated REAMDME.md. Moved lib files. Generated some output documentation.
Other:
- note added: "02-24-2025"
- note added: "Initial Release"
- note added: "NOTE: Jumper for charge current selection"
- note added: "Proto"
Changed lines of the file:
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@@
 	(title_block
 		(title "nRF54L15 ProMicro")
-		(date "2025-02-20")
+		(date "2025-02-24")
 		(rev "Proto")
 		(company "BB Designs")
+	)
+	(text "NOTE: \nJumper for charge current selection"
+		(exclude_from_sim no)
+		(at 44.45 187.452 0)
+		(effects
+			(font
+				(size 1.27 1.27)
+			)
+			(justify left)
+		)
+	)
+	(text "Proto"
+		(exclude_from_sim no)
+		(at 566.166 24.384 0)
+		(effects
+			(font
+				(size 1.27 1.27)
+			)
+		)
 	)
 	(text "Note: VSS_PA to GND PAD ONLY!"
@@
 		)
 	)
+	(text "02-24-2025"
+		(exclude_from_sim no)
+		(at 493.776 24.892 0)
+		(effects
+			(font
+				(size 1.27 1.27)
+			)
+		)
+	)
+	(text "Initial Release"
+		(exclude_from_sim no)
+		(at 527.05 24.638 0)
+		(effects
+			(font
+				(size 1.27 1.27)
+			)
+		)
+	)
 	(text "BLE MCU"
 		(exclude_from_sim no)
-		(at 419.1 93.726 0)
+		(at 421.894 75.946 0)
 		(effects
 			(font

Commit message: BOM updates, schematic and layout updated due to BOM updated
Parts:
- AE1: MFG_PN (none) -> 2450AT18A0100001E
- C13, C14: value 12P -> 9P
- C17, C18: value 12P -> 8P
- D1: MFG (none) -> Harvatek Corporation; MFG_PN (none) -> B18S1UYG-05C000234U1930
- D2: MFG (none) -> Harvatek Corporation; MFG_PN (none) -> B1861NB--05D000134U1930
- J1: MANUFACTURER Amphenol -> (none); MFG (none) -> Amphenol; MFG_PN (none) -> GSB1C4621DS1HR
- L4: footprint Inductor_SMD:L_0402_1005Metric -> Inductor_SMD:L_0603_1608Metric; MFG (none) -> Taiyo Yuden; MFG_PN (none) -> LSCND1608HKT2R2MF
- L5: MFG (none) -> TDK Corporation; MFG_PN (none) -> PLEA67BCA4R7M-1PT00
- L6: value L -> 120R @ 100MHz; footprint Inductor_SMD:L_0402_1005Metric -> Inductor_SMD:L_0201_0603Metric; symbol Device:L -> Device:FerriteBead_Small; MFG (none) -> Murata Electronics; MFG_PN (none) -> BLM03AG121SN1D
- U1: MFG (none) -> Texas Instruments; MFG_PN (none) -> BQ24075RGTR
- U2: value nRF54L10 -> nRF54L15; MFG (none) -> Nordic Semiconductor; MFG_PN (none) -> NRF54L15-QFAA-R; Manufacturer Nordic Semiconductor -> (none)
- U3: MFG (none) -> Texas Instruments; MFG_PN (none) -> TPS62172DSGT
- U4: MFG (none) -> Texas Instruments; MFG_PN (none) -> TPS22917DBVR
- Y1: MFG (none) -> EPSON; MFG_PN (none) -> FC2012SN 32.768K-90NNA0KC0
- Y2: footprint Crystal:Crystal_SMD_2012-2Pin_2.0x1.2mm -> Oscillator:Oscillator_SMD_Abracon_ASCO-4Pin_1.6x1.2mm; symbol Device:Crystal -> Device:Crystal_GND24; MFG (none) -> CTS-Frequency Controls; MFG_PN (none) -> 416F32022CKR
Connections:
- net GND: now also Y2.2, Y2.4
- net XC1: now also Y2.3; no longer Y2.2
Other:
- moved on the sheet: C17, C19, L4

Commit message: BOM Updates. Layout Updates.
Parts:
- AE1: MFG (none) -> Johanson Technology
- C10: MFG (none) -> Murata Electronics; MFG_PN (none) -> GJM1555C1HR30WB01D
- C11, C12, L1, L2, L3: MFG (none) -> Murata Electronics
- R13: value 4.7K -> 1.5K
- R14: value 10K -> 1.5K
Connections:
- net GND: now also U1.6 (EN1); no longer U1.5 (EN2)
- net VSYS renamed 5V5_VSYS
- net 5V5_VSYS: now also U1.5 (EN2); no longer U1.6 (EN1)
Other:
- note added: "03-03-2025"
- note added: "BOM / Schematic Updates"
- note added: "NOTE: Use Internal Rdis"
- note added: "Vf = 1.8V"
- note added: "Vf = 2.7V"
- note removed: "Note: RF GND"
- title: nRF54L15 ProMicro -> nRF54L1x ProMicro
- moved on the sheet: C10, C15, C16, C20, C21, D1, L4, R12, R13, U3, U4

Commit message: Moved USB_D_P/N to MCU Domain for increased bus BW. Improved RF layout. Improved PI. Changed IO for improved MCU escape.
Connections:
- net 3V3_VCC: no longer R1.1
- net USB_D_N: now also U2.11 (P2.00); no longer U2.5 (P1.04)
- net USB_D_P: now also U2.12 (P2.01); no longer U2.4 (P1.03)
- net VEXT_DIS_L: now also U2.8 (P1.07); no longer U2.9 (P1.08)
- net P2.03: now reaches U2.14 (P2.03)
- net P2.03: now also J3.6 (Pin_6)
- net P2.09: now reaches U2.20 (P2.09)
- net P2.09: now also J3.13 (Pin_13)
- net P1.07_AIN3 renamed P1.03
- net P1.03: now also U2.4 (P1.03); no longer U2.8 (P1.07)
- removed net P2.00: J3.6 (Pin_6), U2.11 (P2.00)
- net P2.01_SPI_SCK renamed P2.06_SPI_SCK
- net P2.06_SPI_SCK: now also U2.17 (P2.06); no longer U2.12 (P2.01)
- removed net P2.06: J3.13 (Pin_13), U2.17 (P2.06)
- new net USB_DRV: R1.1, U2.9 (P1.08)
- no-connect marks 14 -> 13
Other:
- note added: "03-10-2025"
- note removed: "03-03-2025"
